File: stDevboard.kicad_pcb (KiCad board)
At the start: 4 copper layers, 0 parts

Commit message: everything I did while on vacation - initial schematic finished, footprints mostly assigned, and pcb layout started
Parts:
- added C1: 22uF, Capacitor_SMD:C_0603_1608Metric, F.Cu at (137.2, 128.8)
- added C10: 1 uF, Capacitor_SMD:C_0603_1608Metric, F.Cu at (137.2, 143.9)
- added C11: 100 nF, Capacitor_SMD:C_0402_1005Metric, F.Cu at (143.5, 134.4)
- added C12: 10 uF, Capacitor_SMD:C_0603_1608Metric, F.Cu at (137.2, 146.4)
- added C13: 100 nF, Capacitor_SMD:C_0402_1005Metric, F.Cu at (143.5, 136.4)
- added C14: 100 nF, Capacitor_SMD:C_0402_1005Metric, F.Cu at (143.5, 138.4)
- added C15: 100 nF, Capacitor_SMD:C_0402_1005Metric, F.Cu at (103.5, 96.0)
- added C16: 2.2uF, Capacitor_SMD:C_0603_1608Metric, F.Cu at (89.6, 109.4)
- added C17: 0.1uF, Capacitor_SMD:C_0402_1005Metric, F.Cu at (103.5, 97.9)
- added C18: 10uF, Capacitor_SMD:C_0603_1608Metric, F.Cu at (89.6, 111.9)
- added C19: 0.1uf, Capacitor_SMD:C_0402_1005Metric, F.Cu at (128.0, 109.3)
- added C2: 10uF, Capacitor_SMD:C_0603_1608Metric, F.Cu at (137.2, 131.3)
- added C20: 2.2uF, Capacitor_SMD:C_0603_1608Metric, F.Cu at (89.6, 114.4)
- added C21: 0.1uF, Capacitor_SMD:C_0402_1005Metric, F.Cu at (103.5, 99.9)
- added C22: 10nF, Capacitor_SMD:C_0402_1005Metric, F.Cu at (103.5, 101.9)
- added C23: 10nF, Capacitor_SMD:C_0402_1005Metric, F.Cu at (103.5, 103.8)
- added C24: 2.2uF, Capacitor_SMD:C_0603_1608Metric, F.Cu at (89.6, 117.0)
- added C25: 0.1uF, Capacitor_SMD:C_0402_1005Metric, F.Cu at (103.5, 105.8)
- added C26: 100uF, Capacitor_SMD:C_0805_2012Metric, F.Cu at (167.6, 156.0)
- added C3: 10 uF, Capacitor_SMD:C_0603_1608Metric, F.Cu at (137.2, 133.8)
- added C4: 100 nF, Capacitor_SMD:C_0402_1005Metric, F.Cu at (143.5, 128.5)
- added C5: 100 nF, Capacitor_SMD:C_0402_1005Metric, F.Cu at (143.5, 130.5)
- added C6: 100 nF, Capacitor_SMD:C_0402_1005Metric, F.Cu at (143.5, 132.5)
- added C7: 1 uF, Capacitor_SMD:C_0603_1608Metric, F.Cu at (137.2, 136.3)
- added C8: 2.2 uF, Capacitor_SMD:C_0603_1608Metric, F.Cu at (137.2, 138.8)
- added C9: 2.2 uF, Capacitor_SMD:C_0603_1608Metric, F.Cu at (137.2, 141.3)
- added D1: D_Zener, Diode_SMD:D_0402_1005Metric, F.Cu at (124.4, 135.8)
- added IC1: MPM3610GQV-Z, footprints:MPM3606GQVZ, F.Cu at (154.6, 100.5)
- added IC2: MMC5603NJ, footprints:MMC5603NJ, F.Cu at (168.8, 121.8)
- added IC3: ICM-42670-P, footprints:ICM42670P, B.Cu at (168.8, 114.8)
- added IC4: MAX-F10S-00B, footprints:MAXF10S00B, F.Cu at (100.2, 128.7)
- added IC5: ICM-45686, footprints:ICM42670P, F.Cu at (168.8, 114.8)
- added IC6: KTS1622EUAA-TR, footprints:KTS1622EUAA-TR, F.Cu at (139.2, 118.0)
- added J9: USB_C_Receptacle_USB2.0_16P, Connector_USB:USB_C_Receptacle_GCT_USB4085, F.Cu at (172.0, 96.0)
- added L1: 2.2 uH, 1.5A, footprints:INDC2520X120N, F.Cu at (181.9, 110.0)
- added Q1: IRLML6402, Package_TO_SOT_SMD:SOT-23, F.Cu at (115.4, 97.2)
- added Q10: IRLML6244, Package_TO_SOT_SMD:SOT-23, F.Cu at (130.1, 97.2)
- added Q11: IRLML6402, Package_TO_SOT_SMD:SOT-23, F.Cu at (130.1, 101.6)
- added Q12: IRLML6244, Package_TO_SOT_SMD:SOT-23, F.Cu at (130.1, 106.1)
- added Q2: IRLML6244, Package_TO_SOT_SMD:SOT-23, F.Cu at (115.4, 101.6)
- added Q3: IRLML6402, Package_TO_SOT_SMD:SOT-23, F.Cu at (115.4, 106.1)
- added Q4: IRLML6244, Package_TO_SOT_SMD:SOT-23, F.Cu at (120.3, 97.2)
- added Q5: IRLML6402, Package_TO_SOT_SMD:SOT-23, F.Cu at (120.3, 101.6)
- added Q6: IRLML6244, Package_TO_SOT_SMD:SOT-23, F.Cu at (120.3, 106.1)
- added Q7: IRLML6402, Package_TO_SOT_SMD:SOT-23, F.Cu at (125.2, 97.2)
- added Q8: IRLML6244, Package_TO_SOT_SMD:SOT-23, F.Cu at (125.2, 101.6)
- added Q9: IRLML6402, Package_TO_SOT_SMD:SOT-23, F.Cu at (125.2, 106.1)
- added R1: 100k, Resistor_SMD:R_0402_1005Metric, F.Cu at (140.6, 128.5)
- added R10: 100, Resistor_SMD:R_0201_0603Metric, F.Cu at (114.2, 109.2)
- added R11: 100, Resistor_SMD:R_0201_0603Metric, F.Cu at (114.2, 110.9)
- added R12: 100, Resistor_SMD:R_0201_0603Metric, F.Cu at (114.2, 112.7)
- added R13: 100, Resistor_SMD:R_0201_0603Metric, F.Cu at (114.2, 114.4)
- added R14: 100, Resistor_SMD:R_0201_0603Metric, F.Cu at (116.6, 109.2)
- added R15: 100, Resistor_SMD:R_0201_0603Metric, F.Cu at (116.6, 110.9)
- added R16: 100, Resistor_SMD:R_0201_0603Metric, F.Cu at (116.6, 112.7)
- added R17: 100, Resistor_SMD:R_0201_0603Metric, F.Cu at (116.6, 114.4)
- added R18: 100, Resistor_SMD:R_0201_0603Metric, F.Cu at (119.1, 109.2)
- added R19: 100, Resistor_SMD:R_0201_0603Metric, F.Cu at (119.1, 110.9)
- added R2: 5.1K, Resistor_SMD:R_0402_1005Metric, F.Cu at (140.6, 130.5)
- added R20: 100, Resistor_SMD:R_0201_0603Metric, F.Cu at (119.1, 112.7)
- added R21: 100, Resistor_SMD:R_0201_0603Metric, F.Cu at (119.1, 114.4)
- added R22: 39k, Resistor_SMD:R_0201_0603Metric, F.Cu at (131.2, 127.5)
- added R23: 75k, Resistor_SMD:R_0201_0603Metric, F.Cu at (131.2, 129.2)
- added R24: 24k, Resistor_SMD:R_0201_0603Metric, F.Cu at (131.2, 131.0)
- added R3: 5.1K, Resistor_SMD:R_0402_1005Metric, F.Cu at (140.6, 132.5)
- added R4: 10k, Resistor_SMD:R_0402_1005Metric, F.Cu at (140.6, 134.5)
- added R5: 10k, Resistor_SMD:R_0402_1005Metric, F.Cu at (140.6, 136.5)
- added R6: 2.7k, Resistor_SMD:R_0402_1005Metric, F.Cu at (98.2, 109.2)
- added R7: 2.7k, Resistor_SMD:R_0402_1005Metric, F.Cu at (98.2, 111.2)
- added R8: 2.7k, Resistor_SMD:R_0402_1005Metric, F.Cu at (140.6, 138.5)
- added R9: 2.7k, Resistor_SMD:R_0402_1005Metric, F.Cu at (140.6, 140.5)
- added U1: STM32, Package_DFN_QFN:QFN-48-1EP_7x7mm_P0.5mm_EP5.6x5.6mm, F.Cu at (180.2, 102.4)
- added U2: BMP581, footprints:BMP581, F.Cu at (159.5, 114.7)
Routing:
- net GND: track 0.00 -> 13.0 mm
- net +5V: track 0.00 -> 7.98 mm
- net Net-(C8-Pad1): track 0.00 -> 4.33 mm
- net Net-(U1-VLXSMPS): track 0.00 -> 4.21 mm
Other:
- board outline added: 50 x 50 mm
