File: pcb/ppu.kicad_sch (KiCad schematic)
At the start: 25 parts, among them IC6 AT25SF041B-SSHB-B, J14 Micro_SD_Card_Det2, Q6 MMBT2222A, U1 STM32U073CCUx, Y4 CM7V-T1A-32.768KHZ

Commit message: added models for some things, fixed micro sd impl and a bunch of other stuff - pcb currently probably ready for production
Parts:
- added R32: 100k, Resistor_SMD:R_0402_1005Metric, symbol Device:R
- renumbered C48 to C50, C49 to C51, C41 to C52, C42 to C53, C44 to C54, C45 to C55, C46 to C56, C47 to C57, C43 to C58, J14 to J10, Q6 to Q8, R32 to R29, R33 to R30, R27 to R31, R28 to R33, R25 to R34, R26 to R35, R31 to R36, U1 to U5
Connections:
- net +3.3V: now also R32.2; no longer J10.9 (DET_B)
- net sd_cs: now reaches J10.2 (DAT3/CD)
- net sd_cs: now also U5.25 (PB12), R32.1
- net sd_det: no longer names the net of J10.10 (DET_A)
- net sd_det: no longer U5.25 (PB12)
- no-connect marks 8 -> 9
